Commit message: replace assets, working non-RL code

File: assets/urdf/dexai/alfred_workstation.urdf (robot description, URDF)
Before this commit: robot alfred_workstation, 6 links, 5 joints
Links:
- removed link low_boy_3pan_west
Joints:
- removed joint low_boy_3pan_with_hotel_pans_to_low_boy_3pan_west
